File: Hardware/PCB/PitotCTRLboard2.brd (EAGLE design)
At the start: 17.8 x 66 mm, 63 parts, among them J1 2201778-1, U1 STM32F405RGT6, U2 MAX1595EUA33+

Commit message: PCB fix
Parts:
- removed R8, R9: 10k, rcl:R0603
- removed SCL1, SCL2, SDA1, SDA2: (no value), wirepad:1,6/0,9
- added CLK, CS1, CS2, SDI, SDO: (no value), wirepad:SMD1,27-2,54
- moved R6 17.5 mm to (-6.35, -10.9), turned to 180 degrees
- moved R7 15.4 mm to (-6.35, -9.02), turned to 180 degrees
- moved G 0.38 mm to (2.16, -17.8)
- moved T+ 0.38 mm to (-2.16, -17.8)
Connections:
- net N$42 renamed INT
- removed net N$40: CHRG.A, U$2.1
- new net N$42: SDO.1, U1.10
- new net N$43: SDI.1, U1.11
- new net N$44: CLK.1, U1.34
- net +3V3: now also R6.1, R7.1; no longer R6.2, R7.2, R8.2, R9.2
- net +5V: now also CHRG.A, U$2.1
- net GND: now also ACCEL.7; no longer TEMP.16
- net N$10: now also R7.2; no longer R6.1, SCL2.1
- net N$11: now also R6.2; no longer R7.1, SDA2.1
- net N$3: now also CS1.1; no longer R8.1, SDA1.1
- net N$4: now also CS2.1; no longer R9.1, SCL1.1
Routing:
- net N$10: track 53.0 -> 24.1 mm
- net N$43: track 0.00 -> 27.3 mm, vias 0 -> 1
- net N$11: track 58.0 -> 30.9 mm
- net N$42: track 0.00 -> 22.9 mm, vias 0 -> 1
- net N$44: track 0.00 -> 18.1 mm, vias 0 -> 1
- net N$3: track 38.7 -> 21.4 mm
- net N$4: track 36.9 -> 19.9 mm
- net N$40: track 11.2 -> 0.00 mm
- net +5V: track 14.8 -> 25.7 mm
- net GND: track 101.2 -> 107.9 mm, vias 9 -> 10
- net N$50: track 33.8 -> 32.1 mm
- net N$32: track 30.1 -> 31.4 mm
- net N$9: track 29.6 -> 30.1 mm
Other:
- board size 17.8 x 66 mm -> 17.8 x 63.6 mm
