File: Hardware/PCB/PitotCTRLboard2.sch (EAGLE design)
At the start: 63 parts, among them J1 2201778-1, U1 STM32F405RGT6, U2 MAX1595EUA33+

Commit message: PCB fix
Parts:
- removed R8, R9: 10k, rcl:R-EU_R0603
- removed SCL1, SCL2, SDA1, SDA2: (no value), wirepad:1,6/0,9
- added CLK, CS1, CS2, SDI, SDO: (no value), wirepad:SMD2
Connections:
- net N$42 renamed INT
- removed net N$40: CHRG.A, U$2.STAT
- new net N$42: SDO.P, U1.PC2/SPI2_MISO
- new net N$43: SDI.P, U1.PC3/SPI2_MOSI
- new net N$44: CLK.P, U1.PB13
- net +3V3: now also R6.1, R7.1; no longer R6.2, R7.2, R8.2, R9.2
- net +5V: now also CHRG.A, U$2.STAT
- net GND: now also ACCEL.RESV_1; no longer TEMP.ADDR
- net N$10: now also R7.2; no longer R6.1, SCL2.P
- net N$11: now also R6.2; no longer R7.1, SDA2.P
- net N$3: now also CS1.P; no longer R8.1, SDA1.P
- net N$4: now also CS2.P; no longer R9.1, SCL1.P
Other:
- moved on the sheet: R6, R7
