File: Hardware/PCB/PitotCTRLboard3.sch (EAGLE design)
At the start: 67 parts, among them J1 2201778-1, U1 STM32F405RGT6, U2 MAX1595EUA33+

Commit message: bug fix
Connections:
- net GND: now also TEMP.ADDR
Changed lines of the file:
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@@
 <junction x="30.48" y="-45.72"/>
 <pinref part="GND3" gate="1" pin="GND"/>
+<pinref part="TEMP" gate="G$1" pin="ADDR"/>
+<wire x1="27.94" y1="-43.18" x2="30.48" y2="-43.18" width="0.1524" layer="91"/>
+<junction x="30.48" y="-43.18"/>
 </segment>
 <segment>
